File: hardware/thermoTester/thermoTester.kicad_pcb (KiCad board)
At the start: 2 copper layers, 147 x 87 mm, 219 parts, among them J10 Power, J20 PRG, J21 YOUT, J22 YOUT, J40 temperature, J41 grating, J42 load, J43 PM9808_TR, J44 XIN, J48 CPTTL, J50 bough, J80 PT100, J81 PT100, Q30 BC817, Q31 BC817, Q32 BC817, Q50 BC817, Q51 BC817, Q52 BC817, Q53 BC807, Q54 BC817, Q55 BC817, Q56 AO3422, U10 XL1509, U11 LM1117-3.3, U20 M_STM32F103RCT6, U21 ULN2003, U22 ULN2003, U40 SP3232, U41 SP3485CN, U50 EL3H4B, U60 EL357N, U61 EL357N, U62 EL357N, U63 EL357N, U64 EL357N, U65 EL357N, U66 EL357N, U80 ADS1220IPWR, U81 CD4051B, U82 CD4051B, U83 CD4051B, Y20 12M

Commit message: 按1.1版本修改硬件和软件代码
Parts:
- added R210: 33k, kicad_footprint_general:R_0603_1608Metric, F.Cu at (65.5, 76.2)
- added R211: 33k, kicad_footprint_general:R_0603_1608Metric, F.Cu at (69.2, 76.2)
- added R212: 33k, kicad_footprint_general:R_0603_1608Metric, F.Cu at (73.1, 76.3)
- added R213: 33k, kicad_footprint_general:R_0603_1608Metric, F.Cu at (76.8, 76.3)
- added R214: 33k, kicad_footprint_general:R_0603_1608Metric, F.Cu at (80.6, 76.3)
- added R215: 33k, kicad_footprint_general:R_0603_1608Metric, F.Cu at (84.3, 76.3)
- added R216: 33k, kicad_footprint_general:R_0603_1608Metric, F.Cu at (88.3, 76.2)
- added R217: 33k, kicad_footprint_general:R_0603_1608Metric, F.Cu at (94.5, 76.2)
- added R218: 33k, kicad_footprint_general:R_0603_1608Metric, F.Cu at (98.4, 76.2)
- added R219: 33k, kicad_footprint_general:R_0603_1608Metric, F.Cu at (102.1, 76.2)
- added R220: 33k, kicad_footprint_general:R_0603_1608Metric, F.Cu at (106.2, 76.2)
- added R221: 33k, kicad_footprint_general:R_0603_1608Metric, F.Cu at (110.2, 76.2)
- added R222: 33k, kicad_footprint_general:R_0603_1608Metric, F.Cu at (114.0, 76.2)
- added R223: 33k, kicad_footprint_general:R_0603_1608Metric, F.Cu at (117.5, 76.2)
- moved D204 26.2 mm to (118.2, 73.9), turned to 180 degrees
- moved D203 24.8 mm to (114.8, 73.9), turned to 180 degrees
- moved D202 23.4 mm to (111.0, 73.9), turned to 180 degrees
- moved D201 21.9 mm to (107.0, 73.9), turned to 180 degrees
- moved D20 21.1 mm to (66.2, 73.9), turned to 180 degrees
- moved D29 20.6 mm to (102.8, 73.9), turned to 180 degrees
- moved D21 20.1 mm to (70.0, 73.9), turned to 180 degrees
- moved D28 19.7 mm to (99.2, 73.9), turned to 180 degrees
- moved D22 19.2 mm to (73.8, 73.9), turned to 180 degrees
- moved D27 18.9 mm to (95.3, 73.9), turned to 180 degrees
- moved D23 18.5 mm to (77.6, 74.0), turned to 180 degrees
- moved D26 18.2 mm to (89.0, 73.9), turned to 180 degrees
- moved D24 18.1 mm to (81.3, 74.0), turned to 180 degrees
- moved D25 18.0 mm to (85.1, 73.9), turned to 180 degrees
- moved U21 3.50 mm to (82.3, 87.8)
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Connections:
- D20 pad 1: Net-(D20-Pad1) -> /Y0
- D20 pad 2: /M_Y0 -> Net-(D20-Pad2)
- D201 pad 1: Net-(D201-Pad1) -> /Y10
- D201 pad 2: /M_Y10 -> Net-(D201-Pad2)
- D202 pad 1: Net-(D202-Pad1) -> /Y11
- D202 pad 2: /M_Y11 -> Net-(D202-Pad2)
- D203 pad 1: Net-(D203-Pad1) -> /Y12
- D203 pad 2: /M_Y12 -> Net-(D203-Pad2)
- D204 pad 1: Net-(D204-Pad1) -> /Y13
- D204 pad 2: /M_Y13 -> Net-(D204-Pad2)
- D21 pad 1: Net-(D21-Pad1) -> /Y1
- D21 pad 2: /M_Y1 -> Net-(D21-Pad2)
- D22 pad 1: Net-(D22-Pad1) -> /Y2
- D22 pad 2: /M_Y2 -> Net-(D22-Pad2)
- D23 pad 1: Net-(D23-Pad1) -> /Y3
- D23 pad 2: /M_Y3 -> Net-(D23-Pad2)
- D24 pad 1: Net-(D24-Pad1) -> /Y4
- D24 pad 2: /M_Y4 -> Net-(D24-Pad2)
- D25 pad 1: Net-(D25-Pad1) -> /Y5
- D25 pad 2: /M_Y5 -> Net-(D25-Pad2)
- D26 pad 1: Net-(D26-Pad1) -> /Y6
- D26 pad 2: /M_Y6 -> Net-(D26-Pad2)
- D27 pad 1: Net-(D27-Pad1) -> /Y7
- D27 pad 2: /M_Y7 -> Net-(D27-Pad2)
- D28 pad 1: Net-(D28-Pad1) -> /Y8
- D28 pad 2: /M_Y8 -> Net-(D28-Pad2)
- D29 pad 1: Net-(D29-Pad1) -> /Y9
- D29 pad 2: /M_Y9 -> Net-(D29-Pad2)
- U21 pad 1: Net-(D20-Pad1) -> /M_Y0
- U21 pad 2: Net-(D21-Pad1) -> /M_Y1
- U21 pad 3: Net-(D22-Pad1) -> /M_Y2
- U21 pad 4: Net-(D23-Pad1) -> /M_Y3
- U21 pad 5: Net-(D24-Pad1) -> /M_Y4
- U21 pad 6: Net-(D25-Pad1) -> /M_Y5
- U21 pad 7: Net-(D26-Pad1) -> /M_Y6
- U22 pad 1: Net-(D27-Pad1) -> /M_Y7
- U22 pad 2: Net-(D28-Pad1) -> /M_Y8
- U22 pad 3: Net-(D29-Pad1) -> /M_Y9
- U22 pad 4: Net-(D201-Pad1) -> /M_Y10
- U22 pad 5: Net-(D202-Pad1) -> /M_Y11
- U22 pad 6: Net-(D203-Pad1) -> /M_Y12
- U22 pad 7: Net-(D204-Pad1) -> /M_Y13
Routing:
- net /VIN: track 133.6 -> 220.6 mm, vias 3 -> 17
- net GND: track 1018.1 -> 1012.3 mm, vias 205 -> 203
- net Net-(D204-Pad1): track 5.30 -> 0.00 mm
- net Net-(D26-Pad1): track 5.21 -> 0.00 mm
- net /Y13: track 33.3 -> 38.3 mm
- net /Y8: track 21.1 -> 26.0 mm
- net /Y12: track 31.3 -> 36.1 mm
- net Net-(D203-Pad1): track 4.78 -> 0.00 mm
- net Net-(D25-Pad1): track 4.76 -> 0.00 mm
- net /Y7: track 18.8 -> 23.5 mm
- net Net-(D202-Pad1): track 4.65 -> 0.00 mm
- net Net-(D27-Pad1): track 4.63 -> 0.00 mm
- net Net-(D24-Pad1): track 4.61 -> 0.00 mm
- net Net-(D20-Pad1): track 4.61 -> 0.00 mm
- net Net-(D201-Pad1): track 4.51 -> 0.00 mm
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Other:
- board text added: "20200811_1.6_HASL"
- board text removed: "20200803_1.6_HASL"

Commit message: 统一sdt_true的定义值，0x01
Connections:
- U80 pad 6: Net-(U80-Pad6) -> GND
Routing:
- net GND: track 1012.3 -> 1013.0 mm
